File: PCB/SupplyMainDigital.sch (KiCad schematic (older format))
At the start: 84 parts, among them CON1 BARREL_JACK, P1 12V, P2 5V, P3 3V3, P4 GND, P5 PGM, P6 SERIAL, P7 I2C, P8 OUT, SW1 SW_PUSH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

Commit message: component layout done
Parts:
- removed TP10, TP11, TP4, TP5: TEST, Measurement_Points:Measurement_Point_Round-SMD-Pad_Small, symbol TEST
- added D4, D5, D6: LED, LEDs:LED_0603, symbol LED
- added R38, R39, R40: 100, Resistors_SMD:R_0603_HandSoldering, symbol R
- C5, C6, C8: footprint Capacitors_Tantalum_SMD:CP_Tantalum_Case-B_EIA-3528-21_Hand -> Capacitors_Tantalum_SMD:CP_Tantalum_Case-A_EIA-3216-18_Reflow
- R14, R15, R16, R17, R18, R19, R20, R21, R22, R23: footprint Resistors_SMD:R_0603_HandSoldering -> Resistors_SMD:R_0805_HandSoldering
Connections:
- net GND: now also D4.1 (K), D5.1 (K), D6.1 (K)
- net SER_RX: now also U5.15 (PGEC2/ASCL2/RP38/RB6), R39.2; no longer U5.12 (CV_REF2O_/RP20/T1CK/RA4)
- net SER_TX: now also U5.16 (SCK1/RP39/INT0/RB7), R38.2; no longer U5.14 (PGED2/ASDA2/RP37/RB5)
- net SPI_CS_DAC: now also U5.12 (CV_REF2O_/RP20/T1CK/RA4); no longer U5.16 (SCK1/RP39/INT0/RB7)
- net SPI_FS: now also U5.14 (PGED2/ASDA2/RP37/RB5); no longer U5.15 (PGEC2/ASCL2/RP38/RB6)
- net at U5.24 (RPI45/CTPLS/RB13): now also R40.1
- new net: D6.2 (A), R40.2
- new net: D5.2 (A), R39.1
- new net: D4.2 (A), R38.1
Other:
- note added: "* Different PIC pins for serial and spi\n* LED's on Serial lines"
- note added: "11/07/2017"
- note added: "V2"

Commit message: Pcb layout V2 ready
Connections:
- net IMON: now also TP9.1, U5.5 (PGEC3/V_REF_+/AN3/OA1OUT/RPI33/CTED1/RB1); no longer TP8.1, U5.4 (PGED3/V_REF_-/AN2/C2IN1-/SS1/RPI32/CTED2/RB0)
- net TEMP: now also TP8.1, U5.4 (PGED3/V_REF_-/AN2/C2IN1-/SS1/RPI32/CTED2/RB0); no longer TP7.1, U5.3 (AN1/C2IN1+/RA1)
- net VSENSE: now also TP7.1, U5.3 (AN1/C2IN1+/RA1); no longer TP9.1, U5.5 (PGEC3/V_REF_+/AN3/OA1OUT/RPI33/CTED1/RB1)
Changed lines of the file:
@@
 Wire Wire Line
 	6050 2650 6700 2650
+Text Label 6300 2050 0    60   ~ 0
+VSENSE
+Text Label 6300 2550 0    60   ~ 0
+TEMP
 Text Label 6300 2650 0    60   ~ 0
-VSENSE
-Text Label 6300 2050 0    60   ~ 0
-TEMP
-Text Label 6300 2550 0    60   ~ 0
 IMON
 Wire Wire Line

Commit message: Pic code for variable with correct output pins
Parts:
- R34: value R -> 2.2k
- U1: symbol TLC272 -> TLC272-RESCUE-SupplyMainDigital
Other:
- note added: "12V DC input"
Changed lines of the file:
@@
 EESchema Schematic File Version 2
+LIBS:SupplyMainDigital-rescue
 LIBS:power
 LIBS:device
@@
 LIBS:contrib
 LIBS:valves
-LIBS:dspic33epxxxgp502
-LIBS:mcp1501
-LIBS:max4080
-LIBS:mcp4131
-LIBS:tlc272
-LIBS:tlv5616c
-LIBS:lt3081
-LIBS:sw_push
-LIBS:lt3080
-LIBS:lm334z
-LIBS:heatsink
 LIBS:SupplyMainDigital-cache
 EELAYER 25 0
@@
 $EndComp
 $Comp
-L TLC272 U1
+L TLC272-RESCUE-SupplyMainDigital U1
 U 2 1 59329EA0
 P 2450 7100
@@
 $EndComp
 $Comp
-L TLC272 U1
+L TLC272-RESCUE-SupplyMainDigital U1
 U 1 1 59329F5F
 P 1000 7000
@@
 P 7750 5100
 F 0 "R34" V 7650 5100 50  0000 C CNN
-F 1 "R" V 7750 5100 50  0000 C CNN
+F 1 "2.2k" V 7750 5100 50  0000 C CNN
 F 2 "Resistors_SMD:R_0603_HandSoldering" V 7680 5100 50  0001 C CNN
 F 3 "" H 7750 5100 50  0000 C CNN
@@
 Wire Wire Line
 	7300 1250 7850 1250
+Text Notes 1300 700  0    60   ~ 0
+12V DC input
 $EndSCHEMATC
