File: PCB/V2/SupplyMainDigital.sch (KiCad schematic (older format))
At the start: 95 parts, among them CON1 BARREL_JACK, P1 12V, P10 GPIO, P2 5V, P3 3V3, P4 GND, P5 PGM, P6 SERIAL, P7 I2C, P8 OUT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

Commit message: next pcb version
Parts:
- R41: value 39k -> 38.3k
Other:
- note added: "LIM"
- note added: "Rlim"
- note added: "Vout"
- moved on the sheet: C10, C12, C14, C2, C22, C23, C4, C6, C7, C9, D3, D7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
