File: PCB/MainController/MainController.kicad_pcb (KiCad board)
At the start: 2 copper layers, 48 parts, among them J1 5V, J2 PGM, J3 SERIAL, J4 I2C, J5 IO, J6 PWR, SW1 SW_Push, SW2 SW, SW3 SW, SW4 SW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

Commit message: pcb lcd
Parts:
- removed REF** (x3): MountingHole_2.7mm_M2.5_ISO14580_Pad, Mounting_Holes:MountingHole_2.7mm_M2.5_ISO14580_Pad
- added J10: Jack-DC, Connect:BARREL_JACK, F.Cu at (139.0, 86.0)
- added J7: MH, Mounting_Holes:MountingHole_2.7mm_M2.5_ISO14580_Pad, F.Cu at (93.0, 50.0)
- added J8: MH, Mounting_Holes:MountingHole_2.7mm_M2.5_ISO14580_Pad, F.Cu at (93.0, 92.0)
- added J9: MH, Mounting_Holes:MountingHole_2.7mm_M2.5_ISO14580_Pad, F.Cu at (151.0, 92.0)
- J1: footprint Connectors_Molex:Molex_PicoBlade_53047-0410_04x1.25mm_Straight -> Pin_Headers:Pin_Header_Straight_1x04_Pitch2.54mm
- SW2, SW3, SW4, SW5: footprint LCD:SW_PUSH_6mm -> LCD:mySW_PUSH_6mm
- SW6: footprint LCD:KSA_Tactile_SPST2 -> LCD:myKSA_Tactile_SPST
- moved C1 31.8 mm to (113.0, 53.0), turned to 180 degrees
- moved D3 16.5 mm to (124.0, 55.0)
- moved C3 16.0 mm to (107.5, 61.0), turned to 90 degrees
- moved D1 15.5 mm to (132.0, 87.0), turned to 90 degrees
- moved C8 14.6 mm to (132.0, 80.0), turned to 270 degrees
- moved R5 14.0 mm to (131.0, 53.0), turned to 180 degrees
- moved D4 13.0 mm to (133.0, 55.0), turned to 180 degrees
- moved R3 12.0 mm to (131.0, 57.0), turned to 180 degrees
- moved C4 11.5 mm to (129.0, 87.0), turned to 90 degrees
- moved C5 11.2 mm to (116.0, 73.0), turned to 180 degrees
- moved D2 11.1 mm to (116.0, 87.0), turned to 90 degrees
- moved U2 11.1 mm to (122.0, 88.0), turned to 90 degrees
- moved R4 11.0 mm to (126.0, 53.0)
- moved U3 11.0 mm to (118.0, 65.0)
- moved J1 9.62 mm to (132.0, 93.0), turned to 270 degrees
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Connections:
- J3 pad 1: (no net) -> Net-(J3-Pad1)
- J5 pad 1: /GPA0 -> /GPA7
- J5 pad 2: /GPA1 -> /GPA6
- J5 pad 3: /GPA2 -> /GPA5
- J5 pad 4: /GPA3 -> /GPA4
- J5 pad 5: /GPA4 -> /GPA3
- J5 pad 6: /GPA5 -> /GPA2
- J5 pad 7: /GPA6 -> /GPA1
- J5 pad 8: /GPA7 -> /GPA0
- J6 pad 3: +5V -> +3V3
- J6 pad 4: +5V -> +3V3
- U1 pad 1: (no net) -> Net-(U1-Pad1)
- U1 pad 2: (no net) -> Net-(U1-Pad2)
- U1 pad 3: (no net) -> Net-(U1-Pad3)
- U3 pad 10: (no net) -> Net-(U3-Pad10)
- U3 pad 2: (no net) -> Net-(U3-Pad2)
- U3 pad 3: (no net) -> Net-(U3-Pad3)
- U3 pad 4: (no net) -> Net-(U3-Pad4)
- U3 pad 9: (no net) -> Net-(U3-Pad9)
- U4 pad 5: (no net) -> Net-(U4-Pad5)
Routing:
- net /IO_INTB: track 0.00 -> 37.3 mm
- net /IO_INTA: track 0.00 -> 35.3 mm
- net /PGM_PGEC: track 0.00 -> 33.7 mm
- net /RESET: track 0.00 -> 33.3 mm
- net /PGM_PGED: track 0.00 -> 32.4 mm
- net /GPA0: track 0.00 -> 28.8 mm
- net /I2C_SCL: track 0.00 -> 27.5 mm, vias 0 -> 4
- net /SER_RX: track 0.00 -> 26.6 mm
- net /GPA1: track 0.00 -> 26.6 mm
- net /GPA2: track 0.00 -> 24.3 mm
- net /SER_TX: track 0.00 -> 23.9 mm
- net /GPA3: track 0.00 -> 22.1 mm
- net /GPA4: track 0.00 -> 19.9 mm
- net /GPA5: track 0.00 -> 17.7 mm
- net /I2C_SDA: track 0.00 -> 17.3 mm
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Other:
- board outline added: 125 x 48 mm

Commit message: pcb lcd
Parts:
- added D5: LED, LEDs:LED_0603_HandSoldering, F.Cu at (136.0, 67.0)
- added D6: LED, LEDs:LED_0603_HandSoldering, F.Cu at (136.0, 65.0)
- added D7: LED, LEDs:LED_0603_HandSoldering, F.Cu at (136.0, 63.0)
- added R14: 2.87k, Resistors_SMD:R_0603_HandSoldering, F.Cu at (131.0, 63.0)
- added R15: 2.87k, Resistors_SMD:R_0603_HandSoldering, F.Cu at (131.0, 65.0)
- added R16: 2.87k, Resistors_SMD:R_0603_HandSoldering, F.Cu at (131.0, 67.0)
- moved D2 21.2 mm to (136.0, 80.0), turned to 270 degrees
- moved R2 17.5 mm to (134.0, 80.0), turned to 90 degrees
- moved C2 5.50 mm to (103.0, 83.5)
- moved C9 2.12 mm to (76.5, 68.5), turned to 270 degrees
- moved C5 1.12 mm to (115.5, 74.0), turned to 270 degrees
Routing:
- net /RESET: track 33.3 -> 103.2 mm, vias 0 -> 4
- net /BTN2: track 0.00 -> 64.1 mm
- net /BTN1: track 0.00 -> 56.4 mm
- net /IO_CS: track 0.00 -> 54.3 mm, vias 0 -> 2
- net /LCD_SS: track 0.00 -> 41.8 mm, vias 0 -> 1
- net GND: track 0.00 -> 40.7 mm, vias 0 -> 26
- net /IO_SDI: track 0.00 -> 40.5 mm
- net /IO_SDO: track 0.00 -> 39.3 mm
- net /IO_SCK: track 0.00 -> 38.0 mm
- net /BTN0: track 0.00 -> 37.6 mm
- net /LCD_SDI: track 0.00 -> 36.9 mm, vias 0 -> 1
- net Net-(R10-Pad2): track 0.00 -> 33.3 mm
- net /LCD_SDO: track 0.00 -> 32.2 mm
- net /LCD_SCK: track 0.00 -> 32.0 mm
- net /BTN3: track 0.00 -> 31.9 mm
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- added copper zone on F.Cu, net +3V3
- added copper zone on F.Cu, net +5V
- added copper zone on B.Cu, net GND
Other:
- board size 125 x 48 mm -> 124 x 48 mm
- board text added: "-"
- board text added: "- GP8"
- board text added: "Button E"
- board text added: "Button N"
- board text added: "Button S"
- board text added: "Button W"
- board text added: "GP1 -"
- board text added: "MCP23S17"
- board text added: "PGM"
- board text added: "Reset"
- board text added: "Turn me on"

Commit message: create main pcb
Parts:
- SW6: footprint LCD:myKSA_Tactile_SPST -> Rotary-Encoders:ALPS_STEC12E08
- moved SW2 2.24 mm to (47.0, 51.5), turned to 180 degrees
- moved SW4 2.24 mm to (47.0, 79.5), turned to 180 degrees
- moved SW5 2.00 mm to (60.0, 65.5)
- moved SW6 1.00 mm to (47.0, 65.5)
Connections:
- J3 pad 1: Net-(J3-Pad1) -> (no net)
- J7 pad 1: Net-(J7-Pad1) -> (no net)
- J8 pad 1: Net-(J8-Pad1) -> (no net)
- J9 pad 1: Net-(J9-Pad1) -> (no net)
- U1 pad 1: Net-(U1-Pad1) -> (no net)
- U1 pad 2: Net-(U1-Pad2) -> (no net)
- U1 pad 3: Net-(U1-Pad3) -> (no net)
- U3 pad 10: Net-(U3-Pad10) -> (no net)
- U3 pad 9: Net-(U3-Pad9) -> (no net)
- U4 pad 5: Net-(U4-Pad5) -> (no net)
Routing:
- net /BTN2: track 64.1 -> 79.2 mm
- net /BTN1: track 56.4 -> 61.2 mm
- net Net-(R12-Pad2): track 16.2 -> 13.4 mm
- net Net-(R11-Pad1): track 29.6 -> 32.3 mm
- net Net-(R10-Pad2): track 33.3 -> 35.8 mm
- net /BTN3: track 31.9 -> 30.6 mm
- net /BTN0: track 37.6 -> 38.7 mm
Other:
- board text removed: "Turn me on"

Commit message: clean up main controller pcb
Parts:
- added G***: Panda, PandaLogos:Panda9x9mm, F.Cu at (144.0, 77.0)
- added J11: MH, Mounting_Holes:MountingHole_2.7mm_M2.5_ISO14580_Pad, F.Cu at (34.0, 81.0)
- added J12: MH, Mounting_Holes:MountingHole_2.7mm_M2.5_ISO14580_Pad, F.Cu at (34.0, 50.0)
Connections:
- J3 pad 1: (no net) -> Net-(J3-Pad1)
- J7 pad 1: (no net) -> Net-(J7-Pad1)
- J8 pad 1: (no net) -> Net-(J8-Pad1)
- J9 pad 1: (no net) -> Net-(J9-Pad1)
- U1 pad 1: (no net) -> Net-(U1-Pad1)
- U1 pad 2: (no net) -> Net-(U1-Pad2)
- U1 pad 3: (no net) -> Net-(U1-Pad3)
- U3 pad 10: (no net) -> Net-(U3-Pad10)
- U3 pad 9: (no net) -> Net-(U3-Pad9)
- U4 pad 5: (no net) -> Net-(U4-Pad5)
Other:
- board text added: "Main controller LCD - UART - I²C V1"
